Commit message: 优化车体模型，debug节点名称错误（暂时没用dae文件）

File: lidarbot_description/urdf/camera.xacro (robot description, xacro)
@@ -1,17 +1,26 @@
 <?xml version="1.0" ?>
 <robot xmlns:xacro="http://ros.org/wiki/xacro">
+  <!-- 【修改点 1】定义参数，用于接收机器人名字 (如 bot1, bot2) -->
+  <xacro:arg name="robot_name" default=""/>
   <!-- Camera -->
   <link name="camera_link">
     <visual>
-      <origin xyz="-0.0115 0.0125 0.0052" rpy="1.8745 ${pi} ${pi/2}"/>
+      <origin xyz="0 0 0" rpy="0 0 0"/>
       <geometry>
-        <mesh filename="package://lidarbot_description/meshes/rpi_camera.dae"/>
+        <box size="0.01 0.03 0.03"/>
       </geometry>
+      <material name="black"/>
     </visual>
+    <collision>
+      <origin xyz="0 0 0" rpy="0 0 0"/>
+      <geometry>
+        <box size="0.01 0.03 0.03"/>
+      </geometry>
+    </collision>
   </link>
   <joint name="camera_joint" type="fixed">
     <parent link="base_link"/>
     <child link="camera_link"/>
-    <origin xyz="0.205 0 0.0425" rpy="0 0 0"/>
+    <origin xyz="0.045 0.015 0.06" rpy="0 0 0"/>
   </joint>
   <link name="camera_link_optical"></link>
@@ -22,23 +31,29 @@
   </joint>
   <gazebo reference="camera_link">
+    <material>Gazebo/Black</material>
     <sensor name="camera" type="camera">
-        <pose> 0 0 0 0 0 0 </pose>
-        <visualize>false</visualize>
-        <update_rate>10</update_rate>
-        <camera>
-            <horizontal_fov>0.934</horizontal_fov>
-            <image>
-                <format>R8G8B8</format>
-                <width>640</width>
-                <height>480</height>
-            </image>
-            <clip>
-                <near>0.05</near>
-                <far>8.0</far>
-            </clip>
-        </camera>
-        <plugin name="camera_controller" filename="libgazebo_ros_camera.so">
-            <frame_name>camera_link_optical</frame_name>
-        </plugin>
+      <pose> 0 0 0 0 0 0 </pose>
+      <visualize>true</visualize>
+      <update_rate>10.0</update_rate>
+      <camera>
+        <horizontal_fov>1.089</horizontal_fov>
+        <image>
+          <format>R8G8B8</format>
+          <width>640</width>
+          <height>480</height>
+        </image>
+        <clip>
+          <near>0.05</near>
+          <far>8.0</far>
+        </clip>
+      </camera>
+      <plugin name="camera_controller" filename="libgazebo_ros_camera.so">
+        <!-- 【修改点 2】关键修复！把机器人名字作为命名空间传入 -->
+        <ros>
+            <namespace>$(arg robot_name)</namespace>
+            <!-- 这样节点就会变成 /bot1/camera_controller 而不是全局冲突 -->
+        </ros>
+        <frame_name>camera_link_optical</frame_name>
+      </plugin>
     </sensor>
   </gazebo>

File: lidarbot_description/urdf/imu.xacro (robot description, xacro)
@@ -1,93 +1,61 @@
 <?xml version="1.0" ?>
 <robot xmlns:xacro="http://ros.org/wiki/xacro">
-  <!-- Imu sensor  -->
-  <link name="imu_link">
-    <visual name="imu_visual">
-      <geometry>
-        <mesh filename="package://lidarbot_description/meshes/MPU6050.dae"/>
-      </geometry>
-    </visual>
-  </link>
-  <joint name="imu_joint" type="fixed">
-    <parent link="base_link"/>
-    <child link="imu_link"/>
-    <origin xyz="0.045 0 0.0175" rpy="0 0 0"/>
-  </joint>
- <gazebo reference="imu_link">
-   <sensor name="mpu6050_imu" type="imu">
-    <plugin name="imu_controller" filename="libgazebo_ros_imu_sensor.so">
-      <frame_name>imu_link</frame_name>
-       <ros>
-         <remapping>~/out:=imu_broadcaster/imu</remapping>
-       </ros>
-      <initial_orientation_as_reference>false</initial_orientation_as_reference>
-    </plugin>
-     <always_on>true</always_on>
-     <!-- Reduced update rate for performance (was 100) -->
-     <update_rate>50</update_rate>
-     <visualize>false</visualize>
-     <imu>
-       <angular_velocity>
-         <x>
-           <noise type="gaussian">
-             <mean>0.0</mean>
-             <stddev>2e-4</stddev>
-           </noise>
-         </x>
-         <y>
-           <noise type="gaussian">
-             <mean>0.0</mean>
-             <stddev>2e-4</stddev>
-           </noise>
-         </y>
-         <z>
-           <noise type="gaussian">
-             <mean>0.0</mean>
-             <stddev>2e-4</stddev>
-           </noise>
-         </z>
-       </angular_velocity>
-       <linear_acceleration>
-         <x>
-           <noise type="gaussian">
-             <mean>0.0</mean>
-             <stddev>1.7e-2</stddev>
-           </noise>
-         </x>
-         <y>
-           <noise type="gaussian">
-             <mean>0.0</mean>
-             <stddev>1.7e-2</stddev>
-           </noise>
-         </y>
-         <z>
-           <noise type="gaussian">
-             <mean>0.0</mean>
-             <stddev>1.7e-2</stddev>
-           </noise>
-         </z>
-       </linear_acceleration>
-       <orientation>
-         <x>
-           <noise type="gaussian">
-              <mean>0.0</mean>
-              <stddev>2e-3</stddev>
-            </noise>
-          </x>
-          <y>
-            <noise type="gaussian">
-              <mean>0.0</mean>
-              <stddev>2e-3</stddev>
-            </noise>
-          </y>
-          <z>
-            <noise type="gaussian">
-              <mean>0.0</mean>
-              <stddev>2e-3</stddev>
-            </noise>
-          </z>
-        </orientation>
-     </imu>
-   </sensor>
- </gazebo>
+    <!-- 【修改点1】接收机器人名字参数 -->
+    <xacro:arg name="robot_name" default=""/>
+    <link name="lidar_link">
+        <visual>
+            <origin xyz="0 0 0" rpy="0 0 0"/>
+            <geometry>
+                <cylinder radius="0.035" length="0.02"/>
+            </geometry>
+            <material name="black">
+                <color rgba="0 0 0 1"/>
+            </material>
+        </visual>
+        <collision>
+            <origin xyz="0 0 0" rpy="0 0 0"/>
+            <geometry>
+                <cylinder radius="0.037" length="0.021"/>
+            </geometry>
+        </collision>
+        <xacro:cylinder_inertia mass="0.1" length="0.021" radius="0.037">
+            <origin xyz="0 0 0" rpy="0 0 0"/>
+        </xacro:cylinder_inertia>
+    </link>
+    <joint name="lidar_joint" type="fixed">
+        <parent link="base_link"/>
+        <child link="lidar_link"/>
+        <origin xyz="0.0 0 0.05" rpy="0 0 0"/>
+    </joint>
+    <gazebo reference="lidar_link">
+        <material>Gazebo/Black</material>
+        <sensor name="lidar" type="ray">
+            <pose> 0 0 0 0 0 0 </pose>
+            <visualize>false</visualize>
+            <update_rate>10</update_rate>
+            <ray>
+                <scan>
+                    <horizontal>
+                        <samples>360</samples>
+                        <resolution>1</resolution>
+                        <min_angle>-3.14</min_angle>
+                        <max_angle>3.14</max_angle>
+                    </horizontal>
+                </scan>
+                <range>
+                    <min>0.3</min>
+                    <max>10</max>
+                </range>
+            </ray>
+            <plugin name="laser_controller" filename="libgazebo_ros_ray_sensor.so">
+                <ros>
+                    <!-- 【修改点2】加入命名空间，解决崩溃的关键！ -->
+                    <namespace>$(arg robot_name)</namespace>
+                    <remapping>~/out:=scan</remapping>
+                </ros>
+                <output_type>sensor_msgs/LaserScan</output_type>
+                <frame_name>lidar_link</frame_name>
+            </plugin>
+        </sensor>
+    </gazebo>
 </robot>

File: lidarbot_description/urdf/lidar.xacro (robot description, xacro)
@@ -1,31 +1,35 @@
 <?xml version="1.0" ?>
 <robot xmlns:xacro="http://ros.org/wiki/xacro">
+    <!-- 【修改点1】接收机器人名字参数 -->
+    <xacro:arg name="robot_name" default=""/>
     <link name="lidar_link">
         <visual>
-            <origin xyz="0 -0.0009 -0.011" rpy="0 0 0"/>
+            <origin xyz="0 0 0" rpy="0 0 0"/>
             <geometry>
-                <mesh filename="package://lidarbot_description/meshes/rplidar_top.dae"/>
+                <cylinder radius="0.035" length="0.02"/>
             </geometry>
+            <material name="black">
+                <color rgba="0 0 0 1"/>
+            </material>
         </visual>
         <collision>
-            <origin xyz="0 -0.0028 0" rpy="0 0 0"/>
+            <origin xyz="0 0 0" rpy="0 0 0"/>
             <geometry>
                 <cylinder radius="0.037" length="0.021"/>
             </geometry>
         </collision>
-         <xacro:cylinder_inertia mass="0.07" length="0.021" radius="0.037">
+        <xacro:cylinder_inertia mass="0.1" length="0.021" radius="0.037">
             <origin xyz="0 0 0" rpy="0 0 0"/>
         </xacro:cylinder_inertia>
-   </link>
+    </link>
     <joint name="lidar_joint" type="fixed">
         <parent link="base_link"/>
         <child link="lidar_link"/>
-        <origin xyz="0.1385 0.0095 0.08" rpy="0 0 ${-pi/2}"/>
-        <axis xyz="0 0 1"/>
+        <origin xyz="0.0 0 0.05" rpy="0 0 0"/>
     </joint>
     <gazebo reference="lidar_link">
+        <material>Gazebo/Black</material>
         <sensor name="lidar" type="ray">
-            <pose>0 0 0 0 0 0</pose>
-            <always_on>true</always_on>
+            <pose> 0 0 0 0 0 0 </pose>
             <visualize>false</visualize>
             <update_rate>10</update_rate>
@@ -34,4 +38,5 @@
                     <horizontal>
                         <samples>360</samples>
+                        <resolution>1</resolution>
                         <min_angle>-3.14</min_angle>
                         <max_angle>3.14</max_angle>
@@ -39,17 +44,12 @@
                 </scan>
                 <range>
-                    <min>0.15</min>
-                    <max>6.0</max>
-                    <!-- <max>12.0</max> -->
-                    <resolution>0.01500</resolution>
-		        </range>
-                <noise>
-                    <type>gaussian</type>
-                    <mean>0.0</mean>
-                    <stddev>0.01</stddev>
-                </noise>
+                    <min>0.3</min>
+                    <max>10</max>
+                </range>
             </ray>
-            <plugin name="lidar_controller" filename="libgazebo_ros_ray_sensor.so">
+            <plugin name="laser_controller" filename="libgazebo_ros_ray_sensor.so">
                 <ros>
+                    <!-- 【修改点2】加入命名空间，解决崩溃的关键！ -->
+                    <namespace>$(arg robot_name)</namespace>
                     <remapping>~/out:=scan</remapping>
                 </ros>

File: lidarbot_description/urdf/lidarbot_core.xacro (robot description, xacro)
@@ -21,8 +21,12 @@
   <link name="base_link">
       <visual>
-        <origin xyz="${base_length/2} 0 ${-wheel_zoff}" rpy="0 0 ${pi}"/>
+        <origin xyz="${base_length/2} 0 ${-wheel_zoff}" rpy="0 0 0"/>
           <geometry>
-              <mesh filename="package://lidarbot_description/meshes/robot_chassis.dae" />
+              <!-- [简化] 使用 Box 代替 Mesh -->
+              <box size="${base_length} ${base_width} ${base_height}"/>
           </geometry>
+          <material name="white">
+            <color rgba="1 1 1 1"/>
+          </material>
       </visual>
       <collision>
@@ -36,6 +40,10 @@
           <origin xyz="0.0185 0 -0.0475" rpy="0 0 0"/>
         <geometry>
-          <mesh filename="package://lidarbot_description/meshes/caster_mount.dae" />
+          <!-- [简化] 使用 Cylinder 代替 Mesh -->
+          <cylinder radius="0.023" length="0.0125"/>
         </geometry>
+        <material name="grey">
+            <color rgba="0.5 0.5 0.5 1"/>
+        </material>
       </visual>
       <collision name="caster_mount_collision">
@@ -47,157 +55,95 @@
       <!-- Rpi stand -->
       <visual name="rpi_4_stand_visual">
-        <origin xyz="0.045 0.015 0.031" rpy="${pi} 0 ${-pi}"/>
+        <origin xyz="0.045 0 0.017" rpy="0 0 0"/>
           <geometry>
-              <mesh filename="package://lidarbot_description/meshes/rpi_stand.dae" />
+             <!-- [简化] 使用 Box 代替 Mesh -->
+             <box size="0.09 0.06 0.03"/>
           </geometry>
+          <material name="black">
+            <color rgba="0 0 0 1"/>
+          </material>
       </visual>
       <collision name="rpi_4_stand_collision">
-        <origin xyz="0.045 0 0.017" rpy="0 0 ${pi/2}"/>
+        <origin xyz="0.045 0 0.017" rpy="0 0 0"/>
         <geometry>
-          <box size="0.098 0.065 0.034"/>
+          <box size="0.09 0.06 0.03"/>
         </geometry>
       </collision>
-      <!-- Raspberry Pi -->
+      <!-- Rpi 4 -->
       <visual name="rpi_4_visual">
-        <origin xyz="0.046 0.00245 0.033" rpy="0 0 ${pi/2}"/>
-        <geometry>
-          <mesh filename="package://lidarbot_description/meshes/rpi_4.dae"/>
-        </geometry>
+        <origin xyz="0.045 0 0.042" rpy="0 0 0"/>
+          <geometry>
+              <!-- [简化] 使用 Box 代替 Mesh -->
+              <box size="0.085 0.056 0.005"/>
+          </geometry>
+          <material name="green">
+            <color rgba="0 0.8 0 1"/>
+          </material>
       </visual>
       <collision name="rpi_4_collision">
-        <origin xyz="0.047 0.005 0.041" rpy="0 0 ${pi/2}"/>
+        <origin xyz="0.045 0 0.042" rpy="0 0 0"/>
         <geometry>
-          <box size="0.09 0.06 0.02"/>
+          <box size="0.085 0.056 0.005"/>
         </geometry>
       </collision>
-      <!-- Power bank stand -->
-      <visual name="power_bank_stand_visual">
-        <origin xyz="0.138 0.015 0.031" rpy="${pi} 0 ${pi}"/>
+      <xacro:box_inertia mass="1.0" length="${base_length}" width="${base_width}" height="${base_height}">
+        <origin xyz="${base_length/2} 0 ${-wheel_zoff}" rpy="0 0 0"/>
+      </xacro:box_inertia>
+  </link>
+  <!-- Robot Footprint -->
+  <link name="base_footprint_link">
+  </link>
+  <joint name="base_footprint_joint" type="fixed">
+    <parent link="base_link"/>
+    <child link="base_footprint_link"/>
+    <origin xyz="0 0 0" rpy="0 0 0"/>
+  </joint>
+  <!-- Wheels -->
+  <xacro:macro name="wheel" params="prefix x_reflect y_reflect">
+    <link name="${prefix}_link">
+      <visual>
+        <origin xyz="0 0 0" rpy="${pi/2} 0 0"/>
         <geometry>
-          <mesh filename="package://lidarbot_description/meshes/power_bank_stand.dae"/>
+            <!-- [简化] 使用 Cylinder 代替 Mesh -->
+            <cylinder radius="${wheel_radius}" length="${wheel_height}"/>
         </geometry>
+        <material name="black">
+            <color rgba="0 0 0 1"/>
+        </material>
       </visual>
-      <collision name="power_bank_stand_collision">
-        <origin xyz="0.138 0 0.0085" rpy="0 0 ${pi/2}"/>
+      <collision>
+        <origin xyz="0 0 0" rpy="${pi/2} 0 0"/>
         <geometry>
-          <box size="0.098 0.065 0.015"/>
+          <cylinder radius="${wheel_radius}" length="${wheel_height}"/>
         </geometry>
       </collision>
-      <!-- Power bank -->
-      <visual name="power_bank_visual">
-        <origin xyz="0.1685 0.04775 0.015" rpy="0 0 ${pi/2}"/>
-        <geometry>
-          <mesh filename="package://lidarbot_description/meshes/power_bank.dae"/>
-        </geometry>
-      </visual>
-      <collision name="power_bank_collision">
-        <origin xyz="0.138 0 0.025" rpy="0 0 ${pi/2}"/>
-        <geometry>
-          <box size="0.096 0.062 0.02"/>
-        </geometry>
-      </collision>
-      <!-- Rplidar stand -->
-      <visual name="rplidar_stand_visual">
-        <origin xyz="0.138 0.015 0.017" rpy="0 0 ${-2*pi}"/>
-        <geometry>
-          <mesh filename="package://lidarbot_description/meshes/rplidar_stand.dae"/>
-        </geometry>
-      </visual>
-      <collision name="rplidar_stand_collision">
-        <origin xyz="0.138 0 0.04" rpy="0 0 ${pi/2}"/>
-        <geometry>
-          <box size="0.098 0.065 0.015"/>
-        </geometry>
-      </collision>
-      <!-- Rplidar base -->
-      <visual name="rplidar_base_visual">
-        <origin xyz="0.13985 0.0087 0.037" rpy="0 0 ${-pi/2}"/>
-          <geometry>
-            <mesh filename="package://lidarbot_description/meshes/rplidar_base.dae"/>
-          </geometry>
-        </visual>
-      <collision name="rplidar_base_collision">
-        <origin xyz="0.138 0 0.056" rpy="0 0 ${-pi/2}"/>
-        <geometry>
-          <box size="0.11 0.072 0.035"/>
-        </geometry>
-      </collision>
-      <!-- Camera mount -->
-      <visual name="camera_mount_visual">
-        <origin xyz="0.16 0.0335 0.001" rpy="0 0 ${pi}"/>
-          <geometry>
-            <mesh filename="package://lidarbot_description/meshes/rpi_camera_mount.dae"/>
-          </geometry>
-      </visual>
-      <collision name="camera_mount_collision">
-        <origin xyz="0.197 0.0 0.032" rpy="${pi/2} 0 ${pi/2}"/>
-        <geometry>
-          <box size="0.048 0.06 0.033"/>
-        </geometry>
-      </collision>
-    <xacro:box_inertia mass="0.864" length="${base_length}" width="${base_width}" height="${base_height}">
-      <origin xyz="0.105 0 0.0175" rpy="0 0 0"/>
-    </xacro:box_inertia>
-  </link>
-  <!-- Left wheel -->
-  <link name="left_wheel">
-    <visual>
-        <geometry>
-          <mesh filename="package://lidarbot_description/meshes/right_wheel.dae" />
-        </geometry>
-    </visual>
-    <collision>
-      <origin xyz="0 0 -0.0065" rpy="0 0 0"/>
-      <geometry>
-        <sphere radius="${wheel_radius}"/>
-      </geometry>
-    </collision>
-    <xacro:cylinder_inertia mass="${wheel_mass}" length="${wheel_height}" radius="${wheel_radius}">
-      <origin xyz="0 0 0" rpy="0 0 0"/>
-    </xacro:cylinder_inertia>
-  </link>
-  <joint name="left_wheel_joint" type="continuous">
-    <parent link="base_link"/>
-    <child link="left_wheel"/>
-    <origin xyz="0.133 0.065 -${wheel_zoff}" rpy="-${pi/2} 0 ${pi}"/>
-    <axis xyz="0 0 -1"/>
-  </joint>
-  <!-- Right wheel -->
-  <link name="right_wheel">
-    <visual>
-      <geometry>
-        <mesh filename="package://lidarbot_description/meshes/right_wheel.dae"/>
-      </geometry>
-    </visual>
-    <collision>
-      <origin xyz="0 0 -0.0065" rpy="0 0 0"/>
-      <geometry>
-        <sphere radius="${wheel_radius}"/>
-      </geometry>
-    </collision>
-    <xacro:cylinder_inertia mass="${wheel_mass}" length="${wheel_height}" radius="${wheel_radius}">
-      <origin xyz="0 0 0" rpy="0 0 0"/>
-    </xacro:cylinder_inertia>
-  </link>
-  <joint name="right_wheel_joint" type="continuous">
-    <parent link="base_link"/>
-    <child link="right_wheel"/>
-    <origin xyz="0.133 -0.065 -${wheel_zoff}" rpy="${pi/2} 0 ${-pi}"/>
-    <axis xyz="0 0 1"/>
-  </joint>
-  <!-- Caster wheel -->
+      <xacro:cylinder_inertia mass="${wheel_mass}" length="${wheel_height}" radius="${wheel_radius}">
+        <origin xyz="0 0 0" rpy="${pi/2} 0 0"/>
+      </xacro:cylinder_inertia>
+    </link>
+    <joint name="${prefix}_joint" type="continuous">
+      <parent link="base_link"/>
+      <child link="${prefix}_link"/>
+      <origin xyz="0 ${y_reflect*0.0725} 0" rpy="0 0 0"/>
+      <axis xyz="0 1 0"/>
+    </joint>
+  </xacro:macro>
+  <xacro:wheel prefix="left_wheel" x_reflect="-1" y_reflect="1" />
+  <xacro:wheel prefix="right_wheel" x_reflect="-1" y_reflect="-1" />
+  <!-- Caster Wheel -->
   <link name="caster_wheel">
     <visual>
       <geometry>
-        <mesh filename="package://lidarbot_description/meshes/caster_wheel.dae"/>
+        <!-- [简化] 使用 Sphere 代替 Mesh -->
+        <sphere radius="0.018"/>
       </geometry>
+      <material name="black"/>
     </visual>
     <collision>
-      <origin xyz="0 0 -0.001" rpy="0 0 ${pi/2}"/>
       <geometry>
-        <sphere radius="0.015"/>
+        <sphere radius="0.018"/>
       </geometry>
     </collision>
-    <xacro:sphere_inertia mass="0.033" radius="0.025">
+    <xacro:sphere_inertia mass="0.01" radius="0.018">
       <origin xyz="0 0 0" rpy="0 0 0"/>
     </xacro:sphere_inertia>
@@ -206,17 +152,23 @@
     <parent link="base_link"/>
     <child link="caster_wheel"/>
-    <origin xyz="0.028 0 -0.031" rpy="0 0 ${pi/2}"/>
+    <origin xyz="0.0185 0 -0.055" rpy="0 0 0"/>
   </joint>
+  <!-- Gazebo Colors -->
+  <gazebo reference="base_link">
+    <material>Gazebo/White</material>
+  </gazebo>
+  <gazebo reference="left_wheel_link">
+    <material>Gazebo/Black</material>
+  </gazebo>
+  <gazebo reference="right_wheel_link">
+    <material>Gazebo/Black</material>
+  </gazebo>
   <gazebo reference="caster_wheel">
+    <material>Gazebo/Black</material>
     <mu1 value="0.001"/>
     <mu2 value="0.001"/>
   </gazebo>
-  <gazebo reference="left_wheel">
-    <mu1 value="1.16"/>
-    <mu2 value="1.16"/>
-  </gazebo>
-  <gazebo reference="right_wheel">
-    <mu1 value="1.16"/>
-    <mu2 value="1.16"/>
+  <gazebo reference="rpi_4_visual">
+    <material>Gazebo/Green</material>
   </gazebo>
 </robot>
