Commit message: 实现了激光雷达扫描建图，尝试合并地图（未完成，使用m-explore-ros2功能包），修正车体模型，仿真摄像头正常工作

File: lidarbot_description/urdf/gazebo_control.xacro (robot description, xacro)
@@ -1,26 +1,26 @@
 <?xml version="1.0" ?>
 <robot xmlns:xacro="http://ros.org/wiki/xacro">
-    <xacro:arg name="robot_name" default="lidarbot"/>
     <gazebo>
-        <plugin name="lidarbot_diff_drive" filename="libgazebo_ros_diff_drive.so">
-            <ros>
-                <namespace>$(arg robot_name)</namespace>
-            </ros>
-            <!-- Wheel information -->
+        <plugin name="diff_drive" filename="libgazebo_ros_diff_drive.so">
+            <!-- Wheel Information -->
             <left_joint>left_wheel_joint</left_joint>
             <right_joint>right_wheel_joint</right_joint>
-            <wheel_separation>0.134</wheel_separation>
-            <wheel_diameter>0.067</wheel_diameter>
-            <!-- Limits (can be adjusted later on)-->
-            <max_wheel_torque>20</max_wheel_torque>
-            <max_wheel_acceleration>2</max_wheel_acceleration>
+            <wheel_separation>0.35</wheel_separation>
+            <wheel_diameter>0.1</wheel_diameter>
+            <!-- Limits -->
+            <max_wheel_torque>200</max_wheel_torque>
+            <max_wheel_acceleration>10.0</max_wheel_acceleration>
             <!-- Output -->
-            <command_topic>cmd_vel</command_topic>
-            <odometry_topic>odom</odometry_topic>
-            <odometry_frame>$(arg robot_name)/odom</odometry_frame>
-            <robot_base_frame>$(arg robot_name)/base_footprint</robot_base_frame>
+            <odometry_source>1</odometry_source>
             <publish_odom>true</publish_odom>
             <publish_odom_tf>true</publish_odom_tf>
             <publish_wheel_tf>true</publish_wheel_tf>
+            <ros>
+                <!-- 关键修改：添加命名空间 -->
+                <namespace>$(arg robot_name)</namespace>
+            </ros>
+            <!-- 关键修改：Frame ID 加上前缀 -->
+            <odometry_frame>$(arg robot_name)/odom</odometry_frame>
+            <robot_base_frame>$(arg robot_name)/base_link</robot_base_frame>
         </plugin>
     </gazebo>

File: lidarbot_description/urdf/imu.xacro (robot description, xacro)
@@ -1,59 +1,41 @@
 <?xml version="1.0" ?>
 <robot xmlns:xacro="http://ros.org/wiki/xacro">
-    <!-- 【修改点1】接收机器人名字参数 -->
-    <xacro:arg name="robot_name" default=""/>
-    <link name="lidar_link">
+    <joint name="imu_joint" type="fixed">
+        <parent link="chassis"/>
+        <child link="imu_link"/>
+        <origin xyz="0 0 0.1" rpy="0 0 0"/>
+    </joint>
+    <link name="imu_link">
         <visual>
-            <origin xyz="0 0 0" rpy="0 0 0"/>
             <geometry>
-                <cylinder radius="0.035" length="0.02"/>
+                <box size="0.05 0.05 0.05"/>
             </geometry>
-            <material name="black">
-                <color rgba="0 0 0 1"/>
-            </material>
+            <material name="black"/>
         </visual>
         <collision>
-            <origin xyz="0 0 0" rpy="0 0 0"/>
             <geometry>
-                <cylinder radius="0.037" length="0.021"/>
+                <box size="0.05 0.05 0.05"/>
             </geometry>
         </collision>
-        <xacro:cylinder_inertia mass="0.1" length="0.021" radius="0.037">
+        <xacro:inertial_box mass="0.1" x="0.05" y="0.05" z="0.05">
             <origin xyz="0 0 0" rpy="0 0 0"/>
-        </xacro:cylinder_inertia>
+        </xacro:inertial_box>
     </link>
-    <joint name="lidar_joint" type="fixed">
-        <parent link="base_link"/>
-        <child link="lidar_link"/>
-        <origin xyz="0.0 0 0.05" rpy="0 0 0"/>
-    </joint>
-    <gazebo reference="lidar_link">
-        <material>Gazebo/Black</material>
-        <sensor name="lidar" type="ray">
-            <pose> 0 0 0 0 0 0 </pose>
-            <visualize>false</visualize>
-            <update_rate>10</update_rate>
-            <ray>
-                <scan>
-                    <horizontal>
-                        <samples>360</samples>
-                        <resolution>1</resolution>
-                        <min_angle>-3.14</min_angle>
-                        <max_angle>3.14</max_angle>
-                    </horizontal>
-                </scan>
-                <range>
-                    <min>0.3</min>
-                    <max>10</max>
-                </range>
-            </ray>
-            <plugin name="laser_controller" filename="libgazebo_ros_ray_sensor.so">
+    <gazebo reference="imu_link">
+        <gravity>true</gravity>
+        <sensor name="imu_sensor" type="imu">
+            <always_on>true</always_on>
+            <update_rate>100</update_rate>
+            <visualize>true</visualize>
+            <topic>__default_topic__</topic>
+            <plugin filename="libgazebo_ros_imu_sensor.so" name="imu_plugin">
                 <ros>
-                    <!-- 【修改点2】加入命名空间，解决崩溃的关键！ -->
+                    <!-- 关键修改：添加命名空间 -->
                     <namespace>$(arg robot_name)</namespace>
-                    <remapping>~/out:=scan</remapping>
+                    <remapping>~/out:=imu</remapping>
                 </ros>
-                <output_type>sensor_msgs/LaserScan</output_type>
-                <frame_name>lidar_link</frame_name>
+                <initial_orientation_as_reference>false</initial_orientation_as_reference>
+                <!-- 关键修改：Frame ID 加上前缀 -->
+                <frame_name>$(arg robot_name)/imu_link</frame_name>
             </plugin>
         </sensor>

File: lidarbot_description/urdf/inertial_macros.xacro (robot description, xacro)
@@ -1,15 +1,21 @@
 <?xml version="1.0" ?>
 <robot xmlns:xacro="http://ros.org/wiki/xacro">
-    <!-- Some standard inertial calculations, obtained from: https://en.wikipedia.org/wiki/List_of_moments_of_inertia -->
-    <xacro:macro name="box_inertia" params="mass length width height *origin">
+    <!-- ================================================== -->
+    <!-- 修正 1: 宏名称改为 inertial_box (配合 imu.xacro) -->
+    <!-- 修正 2: 参数改为 x, y, z (配合 imu.xacro)       -->
+    <!-- ================================================== -->
+    <xacro:macro name="inertial_box" params="mass x y z *origin">
         <inertial>
             <xacro:insert_block name="origin"/>
             <mass value="${mass}"/>
-            <inertia ixx="${(mass/12) * (width*width + height*height)}" ixy="0.0" ixz="0.0"
-                    iyy="${(mass/12) * (length*length + height*height)}" iyz="0.0"
-                    izz="${(mass/12) * (length*length + width*width)}"/>
+            <inertia ixx="${(mass/12) * (y*y + z*z)}" ixy="0.0" ixz="0.0"
+                    iyy="${(mass/12) * (x*x + z*z)}" iyz="0.0"
+                    izz="${(mass/12) * (x*x + y*y)}"/>
         </inertial>
     </xacro:macro>
-    <xacro:macro name="sphere_inertia" params="mass radius *origin">
+    <!-- ================================================== -->
+    <!-- 修正: 宏名称改为 inertial_sphere                    -->
+    <!-- ================================================== -->
+    <xacro:macro name="inertial_sphere" params="mass radius *origin">
         <inertial>
             <xacro:insert_block name="origin"/>
@@ -20,5 +26,8 @@
         </inertial>
     </xacro:macro>
-    <xacro:macro name="cylinder_inertia" params="mass length radius *origin">
+    <!-- ================================================== -->
+    <!-- 修正: 宏名称改为 inertial_cylinder (配合 lidar.xacro) -->
+    <!-- ================================================== -->
+    <xacro:macro name="inertial_cylinder" params="mass length radius *origin">
         <inertial>
             <xacro:insert_block name="origin"/>

File: lidarbot_description/urdf/lidar.xacro (robot description, xacro)
@@ -1,42 +1,36 @@
 <?xml version="1.0" ?>
 <robot xmlns:xacro="http://ros.org/wiki/xacro">
-    <!-- 【修改点1】接收机器人名字参数 -->
-    <xacro:arg name="robot_name" default=""/>
+    <xacro:include filename="inertial_macros.xacro"/>
+    <joint name="laser_joint" type="fixed">
+        <parent link="chassis"/>
+        <child link="lidar_link"/>
+        <origin xyz="0.1 0 0.175" rpy="0 0 0"/>
+    </joint>
     <link name="lidar_link">
         <visual>
-            <origin xyz="0 0 0" rpy="0 0 0"/>
             <geometry>
-                <cylinder radius="0.035" length="0.02"/>
+                <cylinder radius="0.05" length="0.04"/>
             </geometry>
-            <material name="black">
-                <color rgba="0 0 0 1"/>
-            </material>
+            <material name="red"/>
         </visual>
         <collision>
-            <origin xyz="0 0 0" rpy="0 0 0"/>
             <geometry>
-                <cylinder radius="0.037" length="0.021"/>
+                <cylinder radius="0.05" length="0.04"/>
             </geometry>
         </collision>
-        <xacro:cylinder_inertia mass="0.1" length="0.021" radius="0.037">
+        <xacro:inertial_cylinder mass="0.1" length="0.04" radius="0.05">
             <origin xyz="0 0 0" rpy="0 0 0"/>
-        </xacro:cylinder_inertia>
+        </xacro:inertial_cylinder>
     </link>
-    <joint name="lidar_joint" type="fixed">
-        <parent link="base_link"/>
-        <child link="lidar_link"/>
-        <origin xyz="0.0 0 0.05" rpy="0 0 0"/>
-    </joint>
     <gazebo reference="lidar_link">
-        <material>Gazebo/Black</material>
-        <sensor name="lidar" type="ray">
+        <material>Gazebo/Red</material>
+        <sensor name="laser" type="ray">
             <pose> 0 0 0 0 0 0 </pose>
-            <visualize>false</visualize>
-            <update_rate>10</update_rate>
+            <visualize>true</visualize>
+            <update_rate>20</update_rate>
             <ray>
                 <scan>
                     <horizontal>
-                        <samples>360</samples>
-                        <resolution>1</resolution>
+                        <samples>3600</samples>
                         <min_angle>-3.14</min_angle>
                         <max_angle>3.14</max_angle>
@@ -45,15 +39,16 @@
                 <range>
                     <min>0.3</min>
-                    <max>10</max>
+                    <max>12</max>
                 </range>
             </ray>
             <plugin name="laser_controller" filename="libgazebo_ros_ray_sensor.so">
                 <ros>
-                    <!-- 【修改点2】加入命名空间，解决崩溃的关键！ -->
+                    <!-- 关键修改：添加命名空间 -->
                     <namespace>$(arg robot_name)</namespace>
                     <remapping>~/out:=scan</remapping>
                 </ros>
                 <output_type>sensor_msgs/LaserScan</output_type>
-                <frame_name>lidar_link</frame_name>
+                <!-- 关键修改：Frame ID 加上前缀 -->
+                <frame_name>$(arg robot_name)/lidar_link</frame_name>
             </plugin>
         </sensor>

File: lidarbot_description/urdf/lidarbot.urdf.xacro (robot description, xacro)
@@ -1,16 +1,19 @@
 <?xml version="1.0" ?>
-<robot name="lidarbot" xmlns:xacro="http://ros.org/wiki/xacro">
-    <xacro:arg name="use_ros2_control" default="true"/>
-    <xacro:arg name="sim_mode" default="false"/>
-    <xacro:arg name="robot_name" default="lidarbot"/>
+<robot xmlns:xacro="http://ros.org/wiki/xacro" name="lidarbot">
+    <!-- ==================================================== -->
+    <!-- 1. 定义 robot_name 参数 (默认为空，多车时传入 robot1 等) -->
+    <!-- ==================================================== -->
+    <xacro:arg name="robot_name" default=""/>
+    <xacro:include filename="inertial_macros.xacro"/>
     <xacro:include filename="lidarbot_core.xacro"/>
+    <!-- 根据参数选择控制方式 -->
     <xacro:if value="$(arg use_ros2_control)">
-        <xacro:include filename="ros2_control.xacro"/>
+        <xacro:include filename="ros2_control.xacro" />
     </xacro:if>
     <xacro:unless value="$(arg use_ros2_control)">
-        <xacro:include filename="gazebo_control.xacro"/>
+        <xacro:include filename="gazebo_control.xacro" />
     </xacro:unless>
-    <xacro:include filename="camera.xacro"/>
-    <!-- <xacro:include filename="imu.xacro"/> -->
-    <xacro:include filename="lidar.xacro"/>
+    <xacro:include filename="lidar.xacro" />
+    <xacro:include filename="camera.xacro" />
+    <xacro:include filename="imu.xacro" />
 </robot>

File: lidarbot_description/urdf/lidarbot_core.xacro (robot description, xacro)
@@ -1,174 +1,128 @@
 <?xml version="1.0" ?>
 <robot xmlns:xacro="http://ros.org/wiki/xacro">
-  <xacro:include filename="inertial_macros.xacro"/>
-  <!-- Robot's base properties -->
-  <xacro:property name="base_length" value="0.21"/>
-  <xacro:property name="base_width" value="0.11"/>
-  <xacro:property name="base_height" value="0.035"/>
-  <!-- Robot's wheel properties -->
-  <xacro:property name="wheel_radius" value="0.0325"/>
-  <xacro:property name="wheel_height" value="0.025"/>
-  <xacro:property name="wheel_mass" value="0.031"/>
-  <!-- Distance between centre of wheel and robot base -->
-  <xacro:property name="wheel_zoff" value="0.0125"/>
-  <link name="base_footprint"/>
-   <joint name="base_joint" type="fixed">
-     <parent link="base_footprint"/>
-     <child link="base_link"/>
-     <origin xyz="-0.076 0 ${(wheel_radius + wheel_zoff / 2)}" rpy="0 0 0"/>
-   </joint>
-  <!-- Robot base chasis-->
-  <link name="base_link">
-      <visual>
-        <origin xyz="${base_length/2} 0 ${-wheel_zoff}" rpy="0 0 0"/>
-          <geometry>
-              <!-- [简化] 使用 Box 代替 Mesh -->
-              <box size="${base_length} ${base_width} ${base_height}"/>
-          </geometry>
-          <material name="white">
-            <color rgba="1 1 1 1"/>
-          </material>
-      </visual>
-      <collision>
-        <origin xyz="${base_length/2} 0 ${-wheel_zoff}" rpy="0 0 0"/>
-        <geometry>
-          <box size="${base_length} ${base_width} ${base_height}"/>
-        </geometry>
-      </collision>
-    <!-- Caster mount -->
-      <visual name="caster_mount_visual">
-          <origin xyz="0.0185 0 -0.0475" rpy="0 0 0"/>
-        <geometry>
-          <!-- [简化] 使用 Cylinder 代替 Mesh -->
-          <cylinder radius="0.023" length="0.0125"/>
-        </geometry>
-        <material name="grey">
-            <color rgba="0.5 0.5 0.5 1"/>
-        </material>
-      </visual>
-      <collision name="caster_mount_collision">
-        <origin xyz="0.0185 0 -0.005" rpy="0 0 0"/>
-        <geometry>
-          <cylinder radius="0.023" length="0.0125"/>
-        </geometry>
-      </collision>
-      <!-- Rpi stand -->
-      <visual name="rpi_4_stand_visual">
-        <origin xyz="0.045 0 0.017" rpy="0 0 0"/>
-          <geometry>
-             <!-- [简化] 使用 Box 代替 Mesh -->
-             <box size="0.09 0.06 0.03"/>
-          </geometry>
-          <material name="black">
-            <color rgba="0 0 0 1"/>
-          </material>
-      </visual>
-      <collision name="rpi_4_stand_collision">
-        <origin xyz="0.045 0 0.017" rpy="0 0 0"/>
-        <geometry>
-          <box size="0.09 0.06 0.03"/>
-        </geometry>
-      </collision>
-      <!-- Rpi 4 -->
-      <visual name="rpi_4_visual">
-        <origin xyz="0.045 0 0.042" rpy="0 0 0"/>
-          <geometry>
-              <!-- [简化] 使用 Box 代替 Mesh -->
-              <box size="0.085 0.056 0.005"/>
-          </geometry>
-          <material name="green">
-            <color rgba="0 0.8 0 1"/>
-          </material>
-      </visual>
-      <collision name="rpi_4_collision">
-        <origin xyz="0.045 0 0.042" rpy="0 0 0"/>
-        <geometry>
-          <box size="0.085 0.056 0.005"/>
-        </geometry>
-      </collision>
-      <xacro:box_inertia mass="1.0" length="${base_length}" width="${base_width}" height="${base_height}">
-        <origin xyz="${base_length/2} 0 ${-wheel_zoff}" rpy="0 0 0"/>
-      </xacro:box_inertia>
-  </link>
-  <!-- Robot Footprint -->
-  <link name="base_footprint_link">
-  </link>
-  <joint name="base_footprint_joint" type="fixed">
-    <parent link="base_link"/>
-    <child link="base_footprint_link"/>
-    <origin xyz="0 0 0" rpy="0 0 0"/>
-  </joint>
-  <!-- Wheels -->
-  <xacro:macro name="wheel" params="prefix x_reflect y_reflect">
-    <link name="${prefix}_link">
-      <visual>
-        <origin xyz="0 0 0" rpy="${pi/2} 0 0"/>
-        <geometry>
-            <!-- [简化] 使用 Cylinder 代替 Mesh -->
-            <cylinder radius="${wheel_radius}" length="${wheel_height}"/>
-        </geometry>
-        <material name="black">
-            <color rgba="0 0 0 1"/>
-        </material>
-      </visual>
-      <collision>
-        <origin xyz="0 0 0" rpy="${pi/2} 0 0"/>
-        <geometry>
-          <cylinder radius="${wheel_radius}" length="${wheel_height}"/>
-        </geometry>
-      </collision>
-      <xacro:cylinder_inertia mass="${wheel_mass}" length="${wheel_height}" radius="${wheel_radius}">
-        <origin xyz="0 0 0" rpy="${pi/2} 0 0"/>
-      </xacro:cylinder_inertia>
+    <xacro:include filename="inertial_macros.xacro"/>
+    <!-- Robot's base properties -->
+    <xacro:property name="base_length" value="0.21"/>
+    <xacro:property name="base_width" value="0.11"/>
+    <xacro:property name="base_height" value="0.035"/>
+    <!-- Robot's wheel properties -->
+    <xacro:property name="wheel_radius" value="0.05"/>
+    <xacro:property name="wheel_length" value="0.04"/>
+    <xacro:property name="wheel_separation" value="0.35"/>
+    <!-- Robot's caster wheel properties -->
+    <xacro:property name="caster_wheel_radius" value="0.05"/>
+    <xacro:property name="caster_wheel_mass" value="0.1"/>
+    <!-- 🔧 修改点 1: 把万向轮往前移，避免和车身碰撞 (0.15 -> 0.24) -->
+    <xacro:property name="caster_wheel_offset_x" value="0.24"/>
+    <!-- Base Link -->
+    <link name="base_link">
     </link>
-    <joint name="${prefix}_joint" type="continuous">
-      <parent link="base_link"/>
-      <child link="${prefix}_link"/>
-      <origin xyz="0 ${y_reflect*0.0725} 0" rpy="0 0 0"/>
-      <axis xyz="0 1 0"/>
+    <!-- Chassis Link -->
+    <joint name="chassis_joint" type="fixed">
+        <parent link="base_link"/>
+        <child link="chassis"/>
+        <origin xyz="-0.1 0 0"/>
     </joint>
-  </xacro:macro>
-  <xacro:wheel prefix="left_wheel" x_reflect="-1" y_reflect="1" />
-  <xacro:wheel prefix="right_wheel" x_reflect="-1" y_reflect="-1" />
-  <!-- Caster Wheel -->
-  <link name="caster_wheel">
-    <visual>
-      <geometry>
-        <!-- [简化] 使用 Sphere 代替 Mesh -->
-        <sphere radius="0.018"/>
-      </geometry>
-      <material name="black"/>
-    </visual>
-    <collision>
-      <geometry>
-        <sphere radius="0.018"/>
-      </geometry>
-    </collision>
-    <xacro:sphere_inertia mass="0.01" radius="0.018">
-      <origin xyz="0 0 0" rpy="0 0 0"/>
-    </xacro:sphere_inertia>
-  </link>
-  <joint name="caster_wheel_joint" type="fixed">
-    <parent link="base_link"/>
-    <child link="caster_wheel"/>
-    <origin xyz="0.0185 0 -0.055" rpy="0 0 0"/>
-  </joint>
-  <!-- Gazebo Colors -->
-  <gazebo reference="base_link">
-    <material>Gazebo/White</material>
-  </gazebo>
-  <gazebo reference="left_wheel_link">
-    <material>Gazebo/Black</material>
-  </gazebo>
-  <gazebo reference="right_wheel_link">
-    <material>Gazebo/Black</material>
-  </gazebo>
-  <gazebo reference="caster_wheel">
-    <material>Gazebo/Black</material>
-    <mu1 value="0.001"/>
-    <mu2 value="0.001"/>
-  </gazebo>
-  <gazebo reference="rpi_4_visual">
-    <material>Gazebo/Green</material>
-  </gazebo>
+    <link name="chassis">
+        <visual>
+            <origin xyz="0.1 0 0.0175"/>
+            <geometry>
+                <box size="${base_length} ${base_width} ${base_height}"/>
+            </geometry>
+            <material name="white"/>
+        </visual>
+        <collision>
+            <origin xyz="0.1 0 0.0175"/>
+            <geometry>
+                <box size="${base_length} ${base_width} ${base_height}"/>
+            </geometry>
+        </collision>
+        <xacro:inertial_box mass="0.5" x="${base_length}" y="${base_width}" z="${base_height}">
+            <origin xyz="0.1 0 0.0175" rpy="0 0 0"/>
+        </xacro:inertial_box>
+    </link>
+    <!-- 🔧 修改点 2: 给车身添加 Gazebo 材质 -->
+    <gazebo reference="chassis">
+        <material>Gazebo/White</material>
+    </gazebo>
+    <!-- Left Wheel -->
+    <joint name="left_wheel_joint" type="continuous">
+        <parent link="base_link"/>
+        <child link="left_wheel"/>
+        <origin xyz="0 ${wheel_separation/2} 0" rpy="-${pi/2} 0 0"/>
+        <axis xyz="0 0 1"/>
+    </joint>
+    <link name="left_wheel">
+        <visual>
+            <geometry>
+                <cylinder radius="${wheel_radius}" length="${wheel_length}"/>
+            </geometry>
+            <material name="blue"/>
+        </visual>
+        <collision>
+            <geometry>
+                <cylinder radius="${wheel_radius}" length="${wheel_length}"/>
+            </geometry>
+        </collision>
+        <xacro:inertial_cylinder mass="0.1" length="${wheel_length}" radius="${wheel_radius}">
+            <origin xyz="0 0 0" rpy="0 0 0"/>
+        </xacro:inertial_cylinder>
+    </link>
+    <gazebo reference="left_wheel">
+        <material>Gazebo/Blue</material>
+    </gazebo>
+    <!-- Right Wheel -->
+    <joint name="right_wheel_joint" type="continuous">
+        <parent link="base_link"/>
+        <child link="right_wheel"/>
+        <origin xyz="0 -${wheel_separation/2} 0" rpy="${pi/2} 0 0"/>
+        <axis xyz="0 0 -1"/>
+    </joint>
+    <link name="right_wheel">
+        <visual>
+            <geometry>
+                <cylinder radius="${wheel_radius}" length="${wheel_length}"/>
+            </geometry>
+            <material name="blue"/>
+        </visual>
+        <collision>
+            <geometry>
+                <cylinder radius="${wheel_radius}" length="${wheel_length}"/>
+            </geometry>
+        </collision>
+        <xacro:inertial_cylinder mass="0.1" length="${wheel_length}" radius="${wheel_radius}">
+            <origin xyz="0 0 0" rpy="0 0 0"/>
+        </xacro:inertial_cylinder>
+    </link>
+    <gazebo reference="right_wheel">
+        <material>Gazebo/Blue</material>
+    </gazebo>
+    <!-- Caster Wheel -->
+    <joint name="caster_wheel_joint" type="fixed">
+        <parent link="chassis"/>
+        <child link="caster_wheel"/>
+        <origin xyz="${caster_wheel_offset_x} 0 0"/>
+    </joint>
+    <link name="caster_wheel">
+        <visual>
+            <geometry>
+                <sphere radius="${caster_wheel_radius}"/>
+            </geometry>
+            <material name="white"/>
+        </visual>
+        <collision>
+            <geometry>
+                <sphere radius="${caster_wheel_radius}"/>
+            </geometry>
+        </collision>
+        <xacro:inertial_sphere mass="${caster_wheel_mass}" radius="${caster_wheel_radius}">
+            <origin xyz="0 0 0" rpy="0 0 0"/>
+        </xacro:inertial_sphere>
+    </link>
+    <!-- 🔧 修改点 3: 关键！去除万向轮摩擦力，否则车会卡住或乱跳 -->
+    <gazebo reference="caster_wheel">
+        <material>Gazebo/White</material>
+        <mu1 value="0.001"/>
+        <mu2 value="0.001"/>
+    </gazebo>
 </robot>
